File: logger/hardware/logger.kicad_sch (KiCad schematic)
At the start: 44 parts, among them J2 USB_C_Receptacle_USB2.0_14P, J3 S5B-PH-SM4-TB(LF)(SN), J4 Conn_01x04, J5 Micro_SD_Card_Det2, Q1 2N7002K, SW1 SW_Push, SW2 SW_Push, U1 ESP32-S3-WROOM-1-N8, U2 TCAN330, U3 USBLC6-2P6, U4 TPS62172DSG

Commit message: fix: I/O allocations on logger ESP32-S3
Parts:
- U1: value ESP32-S3-WROOM-1-N8 -> ESP32-S3-WROOM-1-N4; LCSC C2913198 -> C2913197
- U3: LCSC C7519 -> C15999
Connections:
- net at J5.8 (DAT1), R11.1: now also U1.10 (IO17); no longer U1.15 (IO3)
Changed lines of the file:
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@@
 	)
 	(junction
-		(at 69.85 106.68)
-		(diameter 0)
-		(color 0 0 0 0)
-	)
-	(junction
 		(at 201.93 132.08)
 		(diameter 0)
@@
 	)
 	(junction
+		(at 69.85 129.54)
+		(diameter 0)
+		(color 0 0 0 0)
+	)
+	(junction
 		(at 152.4 124.46)
 		(diameter 0)
@@
 	(wire
 		(pts
+			(xy 69.85 129.54) (xy 69.85 137.16)
+		)
+		(stroke
+			(width 0)
+			(type default)
+		)
+	)
+	(wire
+		(pts
 			(xy 64.77 134.62) (xy 64.77 137.16)
 		)
@@
 	(wire
 		(pts
+			(xy 130.81 148.59) (xy 130.81 88.9)
+		)
+		(stroke
+			(width 0)
+			(type default)
+		)
+	)
+	(wire
+		(pts
 			(xy 81.28 83.82) (xy 81.28 86.36)
 		)
@@
 	(wire
 		(pts
-			(xy 172.72 107.95) (xy 172.72 91.44)
+			(xy 69.85 129.54) (xy 90.17 129.54)
 		)
 		(stroke
@@
 	(wire
 		(pts
-			(xy 182.88 107.95) (xy 182.88 110.49)
+			(xy 172.72 107.95) (xy 172.72 91.44)
 		)
 		(stroke
@@
 	(wire
 		(pts
-			(xy 30.48 143.51) (xy 30.48 146.05)
+			(xy 182.88 107.95) (xy 182.88 110.49)
 		)
 		(stroke
@@
 	(wire
 		(pts
-			(xy 152.4 111.76) (xy 152.4 114.3)
+			(xy 30.48 143.51) (xy 30.48 146.05)
 		)
 		(stroke
@@
 	(wire
 		(pts
-			(xy 86.36 96.52) (xy 95.25 96.52)
+			(xy 152.4 111.76) (xy 152.4 114.3)
 		)
 		(stroke
@@
 	(wire
 		(pts
-			(xy 69.85 100.33) (xy 69.85 106.68)
-		)
-		(stroke
-			(width 0)
-			(type default)
-		)
-	)
-	(wire
-		(pts
 			(xy 39.37 114.3) (xy 35.56 114.3)
 		)
@@
 		)
 	)
+	(wire
+		(pts
+			(xy 90.17 148.59) (xy 130.81 148.59)
+		)
+		(stroke
+			(width 0)
+			(type default)
+		)
+	)
 	(polyline
 		(pts
@@
 	(wire
 		(pts
-			(xy 69.85 106.68) (xy 69.85 137.16)
+			(xy 69.85 100.33) (xy 69.85 129.54)
 		)
 		(stroke
@@
 	(wire
 		(pts
+			(xy 90.17 129.54) (xy 90.17 148.59)
+		)
+		(stroke
+			(width 0)
+			(type default)
+		)
+	)
+	(wire
+		(pts
 			(xy 57.15 114.3) (xy 95.25 114.3)
 		)
@@
 	(wire
 		(pts
+			(xy 130.81 88.9) (xy 125.73 88.9)
+		)
+		(stroke
+			(width 0)
+			(type default)
+		)
+	)
+	(wire
+		(pts
 			(xy 209.55 129.54) (xy 220.98 129.54)
 		)
@@
 	(wire
 		(pts
-			(xy 86.36 106.68) (xy 86.36 96.52)
-		)
-		(stroke
-			(width 0)
-			(type default)
-		)
-	)
-	(wire
-		(pts
 			(xy 167.64 142.24) (xy 167.64 139.7)
 		)
@@
 	(wire
 		(pts
-			(xy 69.85 106.68) (xy 86.36 106.68)
-		)
-		(stroke
-			(width 0)
-			(type default)
-		)
-	)
-	(wire
-		(pts
 			(xy 205.74 96.52) (xy 205.74 99.06)
 		)
@@
 			)
 		)
-		(property "LCSC" "C7519"
+		(property "LCSC" "C15999"
 			(at 123.19 62.23 0)
 			(hide yes)
@@
 		(dnp no)
 		(property "Reference" "U1"
-			(at 114.554 134.112 0)
+			(at 97.536 79.756 0)
 			(show_name no)
 			(do_not_autoplace no)
@@
 			)
 		)
-		(property "Value" "ESP32-S3-WROOM-1-N8"
-			(at 114.554 136.652 0)
+		(property "Value" "ESP32-S3-WROOM-1-N4"
+			(at 83.566 77.47 0)
 			(show_name no)
 			(do_not_autoplace no)
@@
 			)
 		)
-		(property "LCSC" "C2913198"
+		(property "LCSC" "C2913197"
 			(at 110.49 106.68 0)
 			(hide yes)

Commit message: Logger: Add LEDs, connector silk, layout updates
Parts:
- added D5: GRN, LED_SMD:LED_0603_1608Metric, symbol Device:LED
- added D6: RED, LED_SMD:LED_0603_1608Metric, symbol Device:LED
- added R20, R21: 100, Resistor_SMD:R_0402_1005Metric, symbol Device:R_US
- R4: value 47 -> 100; LCSC C137973 -> C25076
Connections:
- net GND: now also D5.1 (K), D6.1 (K)
- net at U1.38 (IO2): now also R20.1
- net at U1.39 (IO1): now also R21.1
- new net: D5.2 (A), R20.2
- new net: D6.2 (A), R21.2
Other:
- moved on the sheet: C3, C4, C5, C6, J5, R12

Commit message: Logger: Add UART test pads
Parts:
- added TP1: RX, TestPoint:TestPoint_Pad_2.0x2.0mm, symbol Connector:TestPoint
- added TP2: TX, TestPoint:TestPoint_Pad_2.0x2.0mm, symbol Connector:TestPoint
- added TP3: GND, TestPoint:TestPoint_Pad_2.0x2.0mm, symbol Connector:TestPoint
Connections:
- net GND: now also TP3.1
- net at U1.36 (RXD0): now also TP1.1
- net at U1.37 (TXD0): now also TP2.1

Commit message: Logger: Fix GPIO45 usage
Connections:
- net at R16.2, U2.8 (S): now also U1.28 (IO35); no longer U1.26 (IO45)
Changed lines of the file:
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@@
 	(wire
 		(pts
-			(xy 134.62 121.92) (xy 134.62 134.62)
+			(xy 134.62 101.6) (xy 134.62 134.62)
 		)
 		(stroke
@@
 	(wire
 		(pts
-			(xy 125.73 121.92) (xy 134.62 121.92)
-		)
-		(stroke
+			(xy 125.73 101.6) (xy 134.62 101.6)
+		)
+		(stroke

Commit message: Logger: Switch to TPS62162DSGR with 1A output rating
Parts:
- U4: value TPS62172DSG -> TPS62162DSGR; LCSC C59873 -> C40256
Changed lines of the file:
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@@
 			)
 		)
-		(property "Value" "TPS62172DSG"
+		(property "Value" "TPS62162DSGR"
 			(at 212.09 34.29 0)
 			(show_name no)
@@
 			)
 		)
-		(property "LCSC" "C59873"
+		(property "LCSC" "C40256"
 			(at 212.09 46.99 0)
 			(hide yes)
